Commit message: Add files via upload

File: ur3_llm_control/urdf/simple_gripper.urdf.xacro (robot description, xacro)
@@ -5,15 +5,34 @@
       <visual>
         <origin xyz="0 0 0.020" rpy="0 0 0"/>
-        <geometry><box size="0.080 0.120 0.040"/></geometry>
+        <geometry><cylinder radius="0.046" length="0.040"/></geometry>
         <material name="simple_gripper_body"><color rgba="0.18 0.20 0.22 1"/></material>
       </visual>
       <collision>
         <origin xyz="0 0 0.020" rpy="0 0 0"/>
-        <geometry><box size="0.080 0.120 0.040"/></geometry>
+        <geometry><cylinder radius="0.046" length="0.040"/></geometry>
+      </collision>
+      <!-- Small radial ears overlap the round housing and support each finger root. -->
+      <visual>
+        <origin xyz="0 0.043 0.043" rpy="0 0 0"/>
+        <geometry><box size="0.030 0.026 0.020"/></geometry>
+        <material name="simple_gripper_body"/>
+      </visual>
+      <collision>
+        <origin xyz="0 0.043 0.043" rpy="0 0 0"/>
+        <geometry><box size="0.030 0.026 0.020"/></geometry>
+      </collision>
+      <visual>
+        <origin xyz="0 -0.043 0.043" rpy="0 0 0"/>
+        <geometry><box size="0.030 0.026 0.020"/></geometry>
+        <material name="simple_gripper_body"/>
+      </visual>
+      <collision>
+        <origin xyz="0 -0.043 0.043" rpy="0 0 0"/>
+        <geometry><box size="0.030 0.026 0.020"/></geometry>
       </collision>
       <inertial>
         <origin xyz="0 0 0.020" rpy="0 0 0"/>
         <mass value="0.20"/>
-        <inertia ixx="0.00014" ixy="0" ixz="0" iyy="0.00007" iyz="0" izz="0.00016"/>
+        <inertia ixx="0.000133" ixy="0" ixz="0" iyy="0.000133" iyz="0" izz="0.000212"/>
       </inertial>
     </link>
@@ -50,8 +69,31 @@
       </inertial>
     </link>
+    <link name="${prefix}wrist_camera_link">
+      <visual>
+        <origin xyz="0 0 0" rpy="0 0 0"/>
+        <geometry><box size="0.024 0.030 0.014"/></geometry>
+        <material name="wrist_camera_housing"><color rgba="0.12 0.32 0.38 1"/></material>
+      </visual>
+      <visual>
+        <origin xyz="0.013 0 0" rpy="0 1.57079632679 0"/>
+        <geometry><cylinder radius="0.005" length="0.004"/></geometry>
+        <material name="wrist_camera_lens"><color rgba="0.05 0.55 0.95 1"/></material>
+      </visual>
+      <inertial>
+        <origin xyz="0 0 0" rpy="0 0 0"/>
+        <mass value="0.015"/>
+        <inertia ixx="0.000001" ixy="0" ixz="0" iyy="0.000001" iyz="0" izz="0.000001"/>
+      </inertial>
+    </link>
     <joint name="${prefix}simple_gripper_mount_joint" type="fixed">
       <parent link="${parent}"/>
       <child link="${prefix}simple_gripper_base_link"/>
       <origin xyz="0 0 0" rpy="0 0 0"/>
+    </joint>
+    <joint name="${prefix}wrist_camera_joint" type="fixed">
+      <parent link="${prefix}simple_gripper_base_link"/>
+      <child link="${prefix}wrist_camera_link"/>
+      <!-- Aim from the side-mounted lens directly into the jaw gap at the grasp point. -->
+      <origin xyz="0.050 0 0.025" rpy="0 -2.009 0"/>
     </joint>
     <joint name="${prefix}gripper_fixed_finger_joint" type="prismatic">
@@ -60,5 +102,5 @@
       <origin xyz="0 0.045 0.043" rpy="0 0 0"/>
       <axis xyz="0 -1 0"/>
-      <limit lower="0.0" upper="0.015" effort="40" velocity="0.05"/>
+      <limit lower="0.0" upper="0.020" effort="40" velocity="0.05"/>
     </joint>
     <joint name="${prefix}gripper_finger_joint" type="prismatic">
@@ -67,16 +109,31 @@
       <origin xyz="0 -0.045 0.043" rpy="0 0 0"/>
       <axis xyz="0 1 0"/>
-      <limit lower="0.0" upper="0.015" effort="40" velocity="0.05"/>
+      <limit lower="0.0" upper="0.020" effort="40" velocity="0.05"/>
     </joint>
+    <gazebo reference="${prefix}gripper_fixed_finger_link"><mu1>2.0</mu1><mu2>2.0</mu2></gazebo>
+    <gazebo reference="${prefix}gripper_moving_finger_link"><mu1>2.0</mu1><mu2>2.0</mu2></gazebo>
+    <gazebo reference="${prefix}wrist_camera_link">
+      <sensor name="wrist_rgbd" type="rgbd_camera">
+        <pose>0.012 0 0 0 0 0</pose>
+        <always_on>true</always_on>
+        <update_rate>15</update_rate>
+        <topic>/wrist_camera</topic>
+        <camera>
+          <horizontal_fov>0.9599310886</horizontal_fov>
+          <image><width>320</width><height>240</height><format>R8G8B8</format></image>
+          <clip><near>0.02</near><far>1.0</far></clip>
+        </camera>
+      </sensor>
+    </gazebo>
     <xacro:if value="${sim_ignition}">
       <ros2_control name="${prefix}SimpleGripperSystem" type="system">
         <hardware><plugin>ign_ros2_control/IgnitionSystem</plugin></hardware>
         <joint name="${prefix}gripper_finger_joint">
-          <command_interface name="position"><param name="min">0.0</param><param name="max">0.015</param></command_interface>
+          <command_interface name="effort"><param name="min">-40.0</param><param name="max">40.0</param></command_interface>
           <state_interface name="position"><param name="initial_value">0.0</param></state_interface>
           <state_interface name="velocity"/>
         </joint>
         <joint name="${prefix}gripper_fixed_finger_joint">
-          <command_interface name="position"><param name="min">0.0</param><param name="max">0.015</param></command_interface>
+          <command_interface name="effort"><param name="min">-40.0</param><param name="max">40.0</param></command_interface>
           <state_interface name="position"><param name="initial_value">0.0</param></state_interface>
           <state_interface name="velocity"/>

Commit message: Add files via upload

File: ur3_llm_control/urdf/simple_gripper.urdf.xacro (robot description, xacro)
@@ -5,34 +5,15 @@
       <visual>
         <origin xyz="0 0 0.020" rpy="0 0 0"/>
-        <geometry><cylinder radius="0.046" length="0.040"/></geometry>
+        <geometry><box size="0.080 0.120 0.040"/></geometry>
         <material name="simple_gripper_body"><color rgba="0.18 0.20 0.22 1"/></material>
       </visual>
       <collision>
         <origin xyz="0 0 0.020" rpy="0 0 0"/>
-        <geometry><cylinder radius="0.046" length="0.040"/></geometry>
-      </collision>
-      <!-- Small radial ears overlap the round housing and support each finger root. -->
-      <visual>
-        <origin xyz="0 0.043 0.043" rpy="0 0 0"/>
-        <geometry><box size="0.030 0.026 0.020"/></geometry>
-        <material name="simple_gripper_body"/>
-      </visual>
-      <collision>
-        <origin xyz="0 0.043 0.043" rpy="0 0 0"/>
-        <geometry><box size="0.030 0.026 0.020"/></geometry>
-      </collision>
-      <visual>
-        <origin xyz="0 -0.043 0.043" rpy="0 0 0"/>
-        <geometry><box size="0.030 0.026 0.020"/></geometry>
-        <material name="simple_gripper_body"/>
-      </visual>
-      <collision>
-        <origin xyz="0 -0.043 0.043" rpy="0 0 0"/>
-        <geometry><box size="0.030 0.026 0.020"/></geometry>
+        <geometry><box size="0.080 0.120 0.040"/></geometry>
       </collision>
       <inertial>
         <origin xyz="0 0 0.020" rpy="0 0 0"/>
         <mass value="0.20"/>
-        <inertia ixx="0.000133" ixy="0" ixz="0" iyy="0.000133" iyz="0" izz="0.000212"/>
+        <inertia ixx="0.00014" ixy="0" ixz="0" iyy="0.00007" iyz="0" izz="0.00016"/>
       </inertial>
     </link>
@@ -69,31 +50,8 @@
       </inertial>
     </link>
-    <link name="${prefix}wrist_camera_link">
-      <visual>
-        <origin xyz="0 0 0" rpy="0 0 0"/>
-        <geometry><box size="0.024 0.030 0.014"/></geometry>
-        <material name="wrist_camera_housing"><color rgba="0.12 0.32 0.38 1"/></material>
-      </visual>
-      <visual>
-        <origin xyz="0.013 0 0" rpy="0 1.57079632679 0"/>
-        <geometry><cylinder radius="0.005" length="0.004"/></geometry>
-        <material name="wrist_camera_lens"><color rgba="0.05 0.55 0.95 1"/></material>
-      </visual>
-      <inertial>
-        <origin xyz="0 0 0" rpy="0 0 0"/>
-        <mass value="0.015"/>
-        <inertia ixx="0.000001" ixy="0" ixz="0" iyy="0.000001" iyz="0" izz="0.000001"/>
-      </inertial>
-    </link>
     <joint name="${prefix}simple_gripper_mount_joint" type="fixed">
       <parent link="${parent}"/>
       <child link="${prefix}simple_gripper_base_link"/>
       <origin xyz="0 0 0" rpy="0 0 0"/>
-    </joint>
-    <joint name="${prefix}wrist_camera_joint" type="fixed">
-      <parent link="${prefix}simple_gripper_base_link"/>
-      <child link="${prefix}wrist_camera_link"/>
-      <!-- Aim from the side-mounted lens directly into the jaw gap at the grasp point. -->
-      <origin xyz="0.050 0 0.025" rpy="0 -2.009 0"/>
     </joint>
     <joint name="${prefix}gripper_fixed_finger_joint" type="prismatic">
@@ -102,5 +60,5 @@
       <origin xyz="0 0.045 0.043" rpy="0 0 0"/>
       <axis xyz="0 -1 0"/>
-      <limit lower="0.0" upper="0.020" effort="40" velocity="0.05"/>
+      <limit lower="0.0" upper="0.015" effort="40" velocity="0.05"/>
     </joint>
     <joint name="${prefix}gripper_finger_joint" type="prismatic">
@@ -109,31 +67,16 @@
       <origin xyz="0 -0.045 0.043" rpy="0 0 0"/>
       <axis xyz="0 1 0"/>
-      <limit lower="0.0" upper="0.020" effort="40" velocity="0.05"/>
+      <limit lower="0.0" upper="0.015" effort="40" velocity="0.05"/>
     </joint>
-    <gazebo reference="${prefix}gripper_fixed_finger_link"><mu1>2.0</mu1><mu2>2.0</mu2></gazebo>
-    <gazebo reference="${prefix}gripper_moving_finger_link"><mu1>2.0</mu1><mu2>2.0</mu2></gazebo>
-    <gazebo reference="${prefix}wrist_camera_link">
-      <sensor name="wrist_rgbd" type="rgbd_camera">
-        <pose>0.012 0 0 0 0 0</pose>
-        <always_on>true</always_on>
-        <update_rate>15</update_rate>
-        <topic>/wrist_camera</topic>
-        <camera>
-          <horizontal_fov>0.9599310886</horizontal_fov>
-          <image><width>320</width><height>240</height><format>R8G8B8</format></image>
-          <clip><near>0.02</near><far>1.0</far></clip>
-        </camera>
-      </sensor>
-    </gazebo>
     <xacro:if value="${sim_ignition}">
       <ros2_control name="${prefix}SimpleGripperSystem" type="system">
         <hardware><plugin>ign_ros2_control/IgnitionSystem</plugin></hardware>
         <joint name="${prefix}gripper_finger_joint">
-          <command_interface name="effort"><param name="min">-40.0</param><param name="max">40.0</param></command_interface>
+          <command_interface name="position"><param name="min">0.0</param><param name="max">0.015</param></command_interface>
           <state_interface name="position"><param name="initial_value">0.0</param></state_interface>
           <state_interface name="velocity"/>
         </joint>
         <joint name="${prefix}gripper_fixed_finger_joint">
-          <command_interface name="effort"><param name="min">-40.0</param><param name="max">40.0</param></command_interface>
+          <command_interface name="position"><param name="min">0.0</param><param name="max">0.015</param></command_interface>
           <state_interface name="position"><param name="initial_value">0.0</param></state_interface>
           <state_interface name="velocity"/>
